File: thocc-master.kicad_pcb (KiCad board)
At the start: 2 copper layers, 328.6 x 95.3 mm, 170 parts, among them J1 Conn_01x04_Female, J2 Programming Header, U1 AMS1117-3.3, U2 STM32F072CBTx

Commit message: commit
Parts:
- C1: footprint Capacitor_SMD:C_0504_1310Metric_Pad0.83x1.28mm_HandSolder -> Capacitor_SMD:C_0805_2012Metric
- C2, C3, C4, C5, C6, C7: footprint Capacitor_SMD:C_0603_1608Metric -> Capacitor_SMD:C_0805_2012Metric
- moved U1 48.0 mm to (232.6, 108.7), turned to 0 degrees
- moved C3 40.0 mm to (226.8, 109.8), turned to 90 degrees
- moved R1 36.6 mm to (222.8, 116.7)
- moved C2 36.0 mm to (230.1, 116.2), turned to 0 degrees
- moved C5 27.3 mm to (232.6, 127.5), turned to -90 degrees
- moved C1 25.0 mm to (223.7, 133.3), turned to 0 degrees
- moved C4 23.3 mm to (223.7, 131.0)
- moved C6 20.4 mm to (218.9, 117.2), turned to 90 degrees
- moved C7 13.8 mm to (231.9, 130.3)
- moved J2 6.30 mm to (233.6, 144.8)
- moved D52 0.10 mm to (204.4, 140.2)
Connections:
- U2 pad 10: Col11 -> Col3
- U2 pad 11: unconnected-(U2-Pad11) -> Row4
- U2 pad 12: unconnected-(U2-Pad12) -> Row3
- U2 pad 16: Col1 -> Col0
- U2 pad 17: Col0 -> Col1
- U2 pad 18: Row4 -> unconnected-(U2-Pad18)
- U2 pad 19: Row3 -> unconnected-(U2-Pad19)
- U2 pad 2: unconnected-(U2-Pad2) -> Col8
- U2 pad 25: Col12 -> unconnected-(U2-Pad25)
- U2 pad 26: Col13 -> unconnected-(U2-Pad26)
- U2 pad 27: Col14 -> unconnected-(U2-Pad27)
- U2 pad 28: Col15 -> unconnected-(U2-Pad28)
- U2 pad 29: Col2 -> unconnected-(U2-Pad29)
- U2 pad 3: unconnected-(U2-Pad3) -> Col7
- U2 pad 30: Col10 -> unconnected-(U2-Pad30)
- U2 pad 38: unconnected-(U2-Pad38) -> Col2
- U2 pad 39: Col3 -> Col15
- U2 pad 4: unconnected-(U2-Pad4) -> Col6
- U2 pad 40: Col4 -> Col14
- U2 pad 41: Col5 -> Col13
- U2 pad 42: Col6 -> Col12
- U2 pad 43: Col7 -> Col11
- U2 pad 45: Col8 -> Col10
- U2 pad 5: unconnected-(U2-Pad5) -> Col5
- U2 pad 6: unconnected-(U2-Pad6) -> Col4
Routing:
- net Col15: track 78.6 -> 337.3 mm, vias 0 -> 1
- net Col14: track 124.3 -> 373.8 mm
- net Col13: track 45.0 -> 280.5 mm, vias 0 -> 1
- net Col12: track 103.4 -> 326.3 mm
- net Col11: track 100.0 -> 303.6 mm
- net Col10: track 94.3 -> 278.4 mm
- net Col9: track 67.0 -> 231.9 mm
- net Col8: track 67.8 -> 221.0 mm
- net Col7: track 99.0 -> 234.4 mm
- net +3.3V: track 0.00 -> 122.6 mm, vias 0 -> 7
- net Col6: track 67.0 -> 184.0 mm
- net Col5: track 67.0 -> 165.5 mm
- net Row1: track 239.3 -> 332.4 mm
- net Row4: track 253.5 -> 334.3 mm, vias 0 -> 2
- net Col4: track 96.6 -> 176.7 mm
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- added copper zone on B.Cu, net GND
Other:
- outline, holes or cut-outs redrawn

Commit message: The actual keyboard is called voyager
Parts:
- MX17, MX50, MX53, MX65: footprint MX_Only:MXOnly-1U-NoLED -> MX_Only:MXOnly-2U-NoLED
- MX75: footprint MX_Only:MXOnly-1U-NoLED -> MX_Only:MXOnly-6.25U-ReversedStabilizers-NoLED
- MX76: footprint MX_Only:MXOnly-1U-NoLED -> MX_Only:MXOnly-7U-ReversedStabilizers-NoLED
- moved J2 3.26 mm to (230.6, 145.9)
- moved D82 2.43 mm to (493.2, 152.9)
- moved D66 2.40 mm to (493.2, 150.1)
Routing:
- net Net-(J2-Pad3): track 34.6 -> 41.1 mm
- net Net-(J2-Pad1): track 47.2 -> 53.1 mm
- net Row2: track 317.8 -> 322.9 mm
- net GND: track 87.3 -> 91.6 mm
- net Net-(D66-Pad2): track 19.1 -> 23.3 mm
- net Col6: track 184.0 -> 187.4 mm
- net Col3: track 171.8 -> 175.2 mm
- net Col5: track 165.5 -> 168.9 mm
- net Col7: track 234.4 -> 237.8 mm
- net Col4: track 176.7 -> 180.1 mm
- net Col8: track 221.0 -> 224.4 mm
- net Net-(J2-Pad6): track 42.1 -> 39.0 mm
- net Net-(D82-Pad2): track 6.04 -> 8.29 mm
- net +3.3V: track 122.6 -> 124.4 mm
- net Row4: track 334.3 -> 332.8 mm
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