File: thocc-master.kicad_sch (KiCad schematic)
At the start: 170 parts, among them J1 Conn_01x04_Female, J2 Programming Header, U1 AMS1117-3.3, U2 STM32F072CBTx

Commit message: The actual keyboard is called voyager
Parts:
- MX17, MX50, MX53, MX65: footprint MX_Only:MXOnly-1U-NoLED -> MX_Only:MXOnly-2U-NoLED
- MX75: footprint MX_Only:MXOnly-1U-NoLED -> MX_Only:MXOnly-6.25U-ReversedStabilizers-NoLED
- MX76: footprint MX_Only:MXOnly-1U-NoLED -> MX_Only:MXOnly-7U-ReversedStabilizers-NoLED
Changed lines of the file:
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@@
       (effects (font (size 0.508 0.508)))
     )
-    (property "Footprint" "MX_Only:MXOnly-1U-NoLED" (id 2) (at 297.815 101.6 0)
+    (property "Footprint" "MX_Only:MXOnly-2U-NoLED" (id 2) (at 297.815 101.6 0)
       (effects (font (size 1.524 1.524)) hide)
     )
@@
       (effects (font (size 0.508 0.508)))
     )
-    (property "Footprint" "MX_Only:MXOnly-1U-NoLED" (id 2) (at 227.33 118.745 0)
+    (property "Footprint" "MX_Only:MXOnly-6.25U-ReversedStabilizers-NoLED" (id 2) (at 227.33 118.745 0)
       (effects (font (size 1.524 1.524)) hide)
     )
@@
       (effects (font (size 0.508 0.508)))
     )
-    (property "Footprint" "MX_Only:MXOnly-1U-NoLED" (id 2) (at 307.34 50.165 0)
+    (property "Footprint" "MX_Only:MXOnly-2U-NoLED" (id 2) (at 307.34 50.165 0)
       (effects (font (size 1.524 1.524)) hide)
     )
@@
       (effects (font (size 0.508 0.508)))
     )
-    (property "Footprint" "MX_Only:MXOnly-1U-NoLED" (id 2) (at 236.855 118.745 0)
+    (property "Footprint" "MX_Only:MXOnly-7U-ReversedStabilizers-NoLED" (id 2) (at 236.855 118.745 0)
       (effects (font (size 1.524 1.524)) hide)
     )
@@
       (effects (font (size 0.508 0.508)))
     )
-    (property "Footprint" "MX_Only:MXOnly-1U-NoLED" (id 2) (at 158.75 101.6 0)
+    (property "Footprint" "MX_Only:MXOnly-2U-NoLED" (id 2) (at 158.75 101.6 0)
       (effects (font (size 1.524 1.524)) hide)
     )
@@
       (effects (font (size 0.508 0.508)))
     )
-    (property "Footprint" "MX_Only:MXOnly-1U-NoLED" (id 2) (at 307.34 84.455 0)
+    (property "Footprint" "MX_Only:MXOnly-2U-NoLED" (id 2) (at 307.34 84.455 0)
       (effects (font (size 1.524 1.524)) hide)
     )
@@
     )
     (path "/691f833b-93a8-4873-a9ff-b658e7d256a7"
-      (reference "MX17") (unit 1) (value "MX-NoLED") (footprint "MX_Only:MXOnly-1U-NoLED")
+      (reference "MX17") (unit 1) (value "MX-NoLED") (footprint "MX_Only:MXOnly-2U-NoLED")
     )
     (path "/97e26177-e645-4d97-90ab-da5afd021321"
@@
     )
     (path "/bec11edc-bee9-43f9-b8cd-ad7b999c4653"
-      (reference "MX50") (unit 1) (value "MX-NoLED") (footprint "MX_Only:MXOnly-1U-NoLED")
+      (reference "MX50") (unit 1) (value "MX-NoLED") (footprint "MX_Only:MXOnly-2U-NoLED")
     )
     (path "/cd6729da-1a02-4489-86ad-1d576a2648d4"
@@
     )
     (path "/af5eabdc-6016-48bf-9642-a57c1be83371"
-      (reference "MX53") (unit 1) (value "MX-NoLED") (footprint "MX_Only:MXOnly-1U-NoLED")
+      (reference "MX53") (unit 1) (value "MX-NoLED") (footprint "MX_Only:MXOnly-2U-NoLED")
     )
     (path "/892af3ff-0bd7-4acc-9259-caffff63b36e"
@@
     )
     (path "/5ec79c3e-8592-459d-93d2-938d6c545f67"
-      (reference "MX65") (unit 1) (value "MX-NoLED") (footprint "MX_Only:MXOnly-1U-NoLED")
+      (reference "MX65") (unit 1) (value "MX-NoLED") (footprint "MX_Only:MXOnly-2U-NoLED")
     )
     (path "/4f4b7c9c-7d64-4cac-bd37-6f6e3daa79a0"
@@
     )
     (path "/681f2946-ad8d-4ef2-b6e5-96d839aec6ef"
-      (reference "MX75") (unit 1) (value "MX-NoLED") (footprint "MX_Only:MXOnly-1U-NoLED")
+      (reference "MX75") (unit 1) (value "MX-NoLED") (footprint "MX_Only:MXOnly-6.25U-ReversedStabilizers-NoLED")
     )
     (path "/7ed43d20-ca98-425f-b615-60b507f78826"
-      (reference "MX76") (unit 1) (value "MX-NoLED") (footprint "MX_Only:MXOnly-1U-NoLED")
+      (reference "MX76") (unit 1) (value "MX-NoLED") (footprint "MX_Only:MXOnly-7U-ReversedStabilizers-NoLED")
     )
     (path "/1e1eba56-d1f1-4621-b2c2-5e85c77684c8"

Commit message: i hope this isn't a disaster
Other:
- moved on the sheet: D15, D17, D33, D34, D49, D50, D66, MX15, MX18, MX33, MX34, MX49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
